File: Hardware/OpenponicsBoard_Photon_V1.0.brd (EAGLE design)
At the start: 80 x 55.9 mm, 33 parts, among them J1 POWER_JACK, U1 ATLAS_EZO, U2 ATLAS_EZO, U3 BNCPTH, U4 BNCPTH

Commit message: marshall review
Parts:
- added C1: (no value), SparkFun-Capacitors:CPOL-RADIAL-100UF-25V
- moved U$2 16.5 mm to (2.54, -14.0)
- moved U3 16.5 mm to (30.5, -5.08)
- moved U4 16.5 mm to (12.7, -5.08)
- moved U$7 14.3 mm to (22.2, 5.54)
- moved U1 14.0 mm to (30.5, 12.7)
- moved U2 14.0 mm to (12.7, 12.7)
- moved JP1 14.0 mm to (1.27, 8.89)
- moved JP4 14.0 mm to (1.27, 11.4)
- moved U$12 6.54 mm to (48.9, 6.65)
- moved U$9 1.35 mm to (71.8, 2.36)
Connections:
- net GND: now also C1.2
- net VIN: now also C1.1
Routing:
- net 3.3V: track 181.6 -> 194.9 mm
- net TX1: track 64.6 -> 73.6 mm
- net RX1: track 70.1 -> 78.4 mm
- net SCL: track 94.5 -> 99.8 mm
- net SDA: track 98.9 -> 103.6 mm
- net VIN: track 56.7 -> 59.9 mm
- net H2O_TEMP: track 76.7 -> 79.8 mm
- net PRB2: track 6.35 -> 8.89 mm
- net PRB1: track 6.35 -> 8.89 mm
- net PGND2: track 6.35 -> 8.89 mm
- net PGND1: track 6.35 -> 8.89 mm
- net GND: vias 4 -> 8
Other:
- outline, holes or cut-outs redrawn
