File: Hardware/OpenponicsBoard_Photon_V1.0.sch (EAGLE design)
At the start: 24 parts, among them J1 POWER_JACK, U1 ATLAS_EZO, U2 ATLAS_EZO, U3 BNCPTH, U4 BNCPTH

Commit message: marshall review
Parts:
- added C1: (no value), SparkFun-Capacitors:CAP_POLPTH1
Connections:
- net GND: now also C1.-
- net VIN: now also C1.+
Changed lines of the file:
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@@
 <?xml version="1.0" encoding="utf-8"?>
 <!DOCTYPE eagle SYSTEM "eagle.dtd">
-<eagle version="7.3.0">
+<eagle version="7.2.0">
 <drawing>
 <settings>
@@
 <part name="P+5" library="SparkFun" deviceset="VCC" device="" value="3.3V"/>
 <part name="P+3" library="SparkFun" deviceset="VCC" device="" value="3.3V"/>
+<part name="C1" library="SparkFun-Capacitors" deviceset="CAP_POL" device="PTH1"/>
+<part name="GND6" library="SparkFun" deviceset="GND" device=""/>
 </parts>
 <sheets>
@@
 <instance part="SJ1" gate="G$1" x="124.46" y="30.48" rot="R270"/>
 <instance part="GND8" gate="1" x="114.3" y="7.62"/>
-<instance part="GND10" gate="1" x="114.3" y="162.56"/>
+<instance part="GND10" gate="1" x="114.3" y="160.02"/>
 <instance part="P+8" gate="1" x="111.76" y="22.86"/>
 <instance part="P+9" gate="1" x="124.46" y="38.1"/>
@@
 <instance part="SUPPLY3" gate="G$1" x="218.44" y="71.12"/>
 <instance part="F1" gate="G$1" x="119.38" y="175.26"/>
-<instance part="SUPPLY4" gate="G$1" x="129.54" y="177.8"/>
+<instance part="SUPPLY4" gate="G$1" x="137.16" y="177.8"/>
 <instance part="U$13" gate="G$1" x="195.58" y="152.4"/>
 <instance part="P+1" gate="1" x="71.12" y="22.86"/>
 <instance part="P+5" gate="1" x="40.64" y="43.18"/>
 <instance part="P+3" gate="1" x="17.78" y="25.4"/>
+<instance part="C1" gate="G$1" x="132.08" y="170.18"/>
+<instance part="GND6" gate="1" x="132.08" y="160.02"/>
 </instances>
 <busses>
@@
 <pinref part="GND10" gate="1" pin="GND"/>
 <pinref part="J1" gate="G$1" pin="GND"/>
-<wire x1="114.3" y1="165.1" x2="114.3" y2="170.18" width="0.1524" layer="91"/>
+<wire x1="114.3" y1="162.56" x2="114.3" y2="170.18" width="0.1524" layer="91"/>
 <wire x1="114.3" y1="170.18" x2="109.22" y2="170.18" width="0.1524" layer="91"/>
 <pinref part="J1" gate="G$1" pin="GNDBREAK"/>
@@
 <junction x="177.8" y="66.04"/>
 </segment>
+<segment>
+<pinref part="C1" gate="G$1" pin="-"/>
+<pinref part="GND6" gate="1" pin="GND"/>
+<wire x1="132.08" y1="162.56" x2="132.08" y2="165.1" width="0.1524" layer="91"/>
+</segment>
 </net>
 <net name="3.3V" class="0">
@@
 <segment>
 <pinref part="F1" gate="G$1" pin="2"/>
-<wire x1="129.54" y1="175.26" x2="127" y2="175.26" width="0.1524" layer="91"/>
+<wire x1="137.16" y1="175.26" x2="132.08" y2="175.26" width="0.1524" layer="91"/>
 <pinref part="SUPPLY4" gate="G$1" pin="VIN"/>
-<wire x1="129.54" y1="175.26" x2="129.54" y2="177.8" width="0.1524" layer="91"/>
-</segment>
-</net>
+<wire x1="132.08" y1="175.26" x2="127" y2="175.26" width="0.1524" layer="91"/>
+<wire x1="137.16" y1="175.26" x2="137.16" y2="177.8" width="0.1524" layer="91"/>
+<pinref part="C1" gate="G$1" pin="+"/>
+<wire x1="132.08" y1="172.72" x2="132.08" y2="175.26" width="0.1524" layer="91"/>
+<junction x="132.08" y="175.26"/>
+</segment>
+</net>
